File: PMB.sch (EAGLE design)
At the start: 14 parts, among them J1 SOLARP1, J2 SOLARP2, J3 Converter1, J4 Converter2, J5 Battery, J6 ARDUINO, Q1 27W, Q2 27W

Commit message: Add files via upload
Connections:
- removed net N$1: Q2.D
- removed net TRANS1: Q1.S, R1.2
- removed net TRANS2: Q2.S, R3.2
- new net VCC_1: J1.2, Q1.D, R1.2
- new net VCC_2: J3.3, Q1.S
- new net VIN: J4.3, Q2.S
- new net V_BATT: J3.5, J4.5, J5.1
- net VCC: now also Q2.D, R3.2; no longer J1.2, J3.3, J3.5, J4.3, J4.5, J5.1, Q1.D
Other:
- moved on the sheet: J1, J2, J3, J4, J5, J6, Q1, Q2, R3, R4, R5, R6
