File: PMB_LED.sch (EAGLE design)
At the start: 21 parts, among them J1 SOLARP1, J10 PWL3, J2 SOLARP2, J3 Converter1, J4 Converter2, J5 Battery_out, J6 Battery_in, J7 2X6 FEMALE, J8 PWL2, J9 PWL1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

Commit message: Add files via upload
Parts:
- J10: value PWL3 -> ARDUINO; device SparkFun-Connectors:CONN_02LOCK_LONGPADS -> SparkFun-Connectors:CONN_06X2PTH_FEMALE
- J5: value Battery_out -> Battery_charge
- J6: value Battery_in -> Battery_input
- J7: value 2X6 FEMALE -> (none); device SparkFun-Connectors:CONN_06X2PTH_FEMALE -> SparkFun-Connectors:CONN_02
- J8: value PWL2 -> (none); device SparkFun-Connectors:CONN_02LOCK_LONGPADS -> SparkFun-Connectors:CONN_02
- J9: value PWL1 -> (none); device SparkFun-Connectors:CONN_02LOCK_LONGPADS -> SparkFun-Connectors:CONN_02
- Q3, Q4, Q5: value 7W -> 27W; device SparkFun-DiscreteSemi:MOSFET-NCH-AO3404A -> SparkFun-DiscreteSemi:MOSFET-NCH-FDD8780
- R1, R3: value 220k -> 220K
- R2, R4: value 620k -> 620K
Connections:
- removed net N$4: J10.1, Q5.D
- removed net TRANS1: Q1.S, R1.2
- removed net TRANS2: Q2.S, R3.2
- new net VCC_1: J1.2, Q1.D, R1.2
- new net VCC_2: J3.3, Q1.S
- new net VDD: J6.1, J7.2, J8.2, J9.2
- new net VIN: J4.3, Q2.S
- new net V_BATT: J3.5, J4.5, J5.1
- net !SHDN3: now also J10.8; no longer J7.2
- net !SHDN4: now also J10.10; no longer J7.4
- net ARDU_CHECK3: now also J10.1; no longer J7.5
- net ARDU_CHECK4: now also J10.2; no longer J7.6
- net ARDU_SWITCH3: now also J10.3; no longer J7.7
- net ARDU_SWITCH4: now also J10.4; no longer J7.8
- net ARDU_SWITCH5: now also J10.5, Q4.G; no longer J7.9, Q3.G
- net ARDU_SWITCH6: now also J10.6, Q3.G; no longer J7.10, Q4.G
- net ARDU_SWITCH7: now also J10.7; no longer J7.11
- net GND: now also J10.12, Q3.D, Q4.D, Q5.D; no longer J7.12, Q3.S, Q4.S, Q5.S
- net N$1: now also J8.1, Q3.S; no longer Q2.D
- net N$2: now also Q5.S; no longer Q3.D
- net N$3: now also J7.1, Q4.S; no longer J8.1, Q4.D
- net PG3: now also J10.9; no longer J7.1
- net PG4: now also J10.11; no longer J7.3
- net VCC: now also Q2.D, R3.2; no longer J1.2, J10.2, J3.3, J3.5, J4.3, J4.5, J5.1, J6.1, J8.2, J9.2, Q1.D
Other:
- moved on the sheet: J1, J2, J3, J4, J5, J6, J8, J9, Q1, Q2, Q3, Q4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
