File: astronaut_mainboard_2.sch (EAGLE design)
At the start: 32 parts, among them IC1 ADUM1250, IC2 741G3157DBVR, IC3 741G3157DBVR, J1 User Interface (I2C), J2 Arduino Mega (UART), J3 HF Comm (UART), J4 User Interface (I2C), J5 GNSS (UART), Q1 BSS138, Q2 BSS138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

Commit message: minor updates
Parts:
- removed J1: User Interface (I2C), EP_molex_6410_7395:22-05-7048-04
- removed Q2, Q4: BSS138, SparkFun-DiscreteSemi:MOSFET-NCH-AO3404A
- removed R1, R15, R16, R2: 470, rcl:R-EU_R0805
- removed R10, R5, R8, R9: 10k, rc-master-smd:R_1206
Connections:
- removed net ARDU_PIN_3: J1-2.S, Q2.D, R15.1, R8.1
- removed net ARDU_PIN_4: J1-3.S, Q4.D, R10.1, R16.1
- net +5V: no longer J1-1.S, R10.2, R15.2, R16.2, R8.2
- net GND: no longer J1-4.S
- net I2C2_SCL: no longer Q4.S, R2.1, R9.1
- net I2C2_SDA: no longer Q2.S, R1.1, R5.1
- net VCC: no longer Q2.G, Q4.G, R1.2, R2.2, R5.2, R9.2
Other:
- note removed: "select with/without galvanic isolation"
- moved on the sheet: IC1, IC2, IC2P, IC3, IC3P, J2-1, J2-2, J2-3, J2-4, J3-1, J3-2, J3-3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

Commit message: added boards for astronaut
Parts:
- removed R6, R7: 10k, rc-master-smd:R_1206
- removed U$1: NUCLEO_F411RE, stm32_nucleo_shield:NUCLEO_F411RE
- added J1: EXT_SUPP, EP_molex_6410_7395:22-05-7028-02
- added JP1: (no value), pinhead:PINHD-1X2
- added R1, R2: 10k, rcl:R-EU_R0805
- added U$3: NUCLEO_F411RE_MORPHO, stm32_nucleo_shield:NUCLEO_F411RE_MORPHO
- R3, R4: device rc-master-smd:R_1206 -> rcl:R-EU_R0805
Connections:
- net VDD renamed VEE
- new net E5V: JP1.1, U$3G$1.E5V
- net +5V: now also J1-2.S, JP1.2, R1.2, R3.2, U$3G$1.5V@1; no longer R4.2, R7.2, U$1G$2.5V@1
- net ARDU_PIN_1: now also R1.1; no longer R7.1
- net ARDU_PIN_2: now also R3.1; no longer R4.1
- net GND: now also J1-1.S, U$3G$1.GND@3, U$3G$1.GND@4; no longer U$1G$2.GND@3, U$1G$2.GND@4
- net I2C2_SCL: now also U$3G$2.PB4@1; no longer U$1G$3.PB10@1
- net I2C2_SDA: now also U$3G$2.AVDD@1; no longer U$1G$3.PB9@1
- net LED_DGB: now also U$3G$2.PB3@1; no longer U$1G$3.PB5@1
- net USART1_RX: now also U$3G$2.PA2@1; no longer U$1G$1.PA10@10
- net USART1_TX: now also U$3G$2.PA8@1; no longer U$1G$1.PA9@10
- net USART6_RX: now also U$3G$2.PA9@1; no longer U$1G$3.PC7@1
- net USART6_RX_A: now also R2.1; no longer R6.1
- net USART6_SEL: now also U$3G$2.PC7@1; no longer U$1G$3.PB6@1
- net USART6_TX: now also U$3G$2.PC5; no longer U$1G$3.PC6
- net USART6_TX_A: now also R4.1; no longer R3.1
- net VCC: now also R2.2, R4.2, U$3G$1.3V3@1; no longer R3.2, R6.2, U$1G$2.3V3@1
