File: gs_mainboard.sch (EAGLE design)
At the start: 24 parts, among them IC1 LM4040, J1 22-05-7028-02, J2 LF Comm, J4 HF Comm (UART)

Commit message: minor updates
Parts:
- removed R29: 220, rcl:R-EU_M0805
- removed U$2: AM1S-0505, am1s:AM1S-0505
- added D3, D4: 4,7V, diode:ZENER-DIODEDO35Z10
- added IC2: LM358N, linear:LM358N
- added J5: Weather station (SPI), EP_molex_6410_7395:22-05-7068-06
- added Q1, Q2, Q3, Q4: BSS138, SparkFun-DiscreteSemi:MOSFET-NCH-AO3404A
- added R10, R11, R12, R13, R14, R15, R16, R9: 10k, rc-master-smd:R_1206
- added R7: 5k6, rcl:R-EU_R0805
- added R8: 2k, rcl:R-EU_R0805
- IC1: value LM4040 -> LM4040/385 (2.5V)
- R1: value 1k2 -> 5k6
- R2: value 1k -> 2k
- R27, R3: value 220 -> 470
Connections:
- removed net GND2: J2-4.S, R4.1, U$2.V-OUT
- removed net I2C2_SDA: U$1G$3.PB9@1
- removed net N$22: OK1.COL, R29.1
- removed net SS: R27.2
- removed net USART6_RX: U$1G$3.PC7@1
- removed net USART6_TX: U$1G$3.PC6
- removed net VDD: R5.2, R6.2, U$2.V+OUT
- new net LF_TX1: IC2A.+IN, OK2.EMIT, R4.2, R6.1
- new net N$2: R7.1, R8.2, U$13.CH1
- new net N$4: D3.A, D4.C
- new net SPI2_SS: R27.2, U$1G$2.PC1@1
- new net SPI3_MISO: Q1.S, R11.1, U$1G$2.PC11
- new net SPI3_MISO_EXT: J5-3.S, Q1.D, R12.1
- new net SPI3_MOSI: Q3.S, R9.1, U$1G$2.PC12
- new net SPI3_MOSI_EXT: J5-2.S, Q3.D, R10.1
- new net SPI3_SCK: Q2.S, R13.1, U$1G$3.PB12
- new net SPI3_SS: Q4.S, R15.1, U$1G$3.PC9
- new net SPI3_SS_EXT: J5-4.S, Q2.D, R14.1
- new net SPI3_SS_EXT1: J5-5.S, Q4.D, R16.1
- net +5V: now also J5-1.S, R10.2, R12.2, R14.2, R16.2, U$1G$1.5V@10; no longer U$2.V+IN
- net GND: now also J5-6.S; no longer U$2.V-IN
- net GND1: now also D4.A, IC2P.V-, J2-4.S, R4.1, R8.1, U$13.CH2, U$13.CH3, U$13.CH4, U$13.CH5, U$13.CH6, U$13.CH7
- net LF_RX: now also D3.C, R7.2
- net LF_TX: now also IC2A.-IN, IC2A.OUT; no longer OK2.EMIT, R4.2, R6.1
- net LF_TX_UC: now also U$1G$3.PC6
- net VCC: now also Q1.G, Q2.G, Q3.G, Q4.G, R11.2, R13.2, R15.2, R9.2
- net VEE: now also IC2P.V+, OK1.COL, R5.2, R6.2; no longer R29.2
Other:
- note added: "UART1 (HF) SPI2 (LF)(ADC) SPI2 (storm detector)(ADC) SPI3 (weather station)"
- note added: "wątpliwości co do odbioru radia?"
- note removed: "EJ, JAK CHCEMY ODBIERAĆ TO RADIO? :D"
- note removed: "UART (LF) UART (HF) ?? storm detector +POWER (USB?)"
- note removed: "dodac brakujace gpio"
- note removed: "w ogole jak to przestrzennie umiescic wszystkie rzeczy? moze dwm i cos na jednej plytce?"
- moved on the sheet: C2, D1, D2, IC1, J1-1, J1-2, J2-1, J2-2, J2-3, J2-4, J4-1, J4-2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

Commit message: added gs_mainboard layout
Parts:
- removed D2, D4: 4,7V, diode:ZENER-DIODEDO35Z10
- removed R16: 10k, rc-master-smd:R_1206
- removed U$1: NUCLEO_F411RE, stm32_nucleo_shield:NUCLEO_F411RE
- added J3: EXT_SUPP, EP_molex_6410_7395:22-05-7028-02
- added JP1: (no value), pinhead:PINHD-1X2
- added R17: 10k, rcl:R-EU_M0805
- added U$2: NUCLEO_F411RE_MORPHO, stm32_nucleo_shield:NUCLEO_F411RE_MORPHO
- D1, D3: value 4,7V -> 9V; device diode:ZENER-DIODEDO35Z10 -> diode:ZENER-DIODESOD80C
- IC2: value LM358N -> LM358D; device linear:LM358N -> linear:LM358D
- J1: value 22-05-7028-02 -> Storm Det
- R10, R11, R12, R13, R14, R15, R9: device rc-master-smd:R_1206 -> rcl:R-EU_M0805
- U$13: value MCP3008P -> MCP3008SL; device MCP300x:MCP3008P -> MCP300x:MCP3008SL
Connections:
- removed net N$1: D1.A, D2.C
- removed net N$4: D3.A, D4.C
- new net E5V: JP1.1, U$2G$1.E5V
- net +5V: now also J3-2.S, JP1.2, R11.2, R13.2, R15.2, R9.2, U$2G$1.5V@1; no longer R10.2, R12.2, R14.2, R16.2, U$1G$1.5V@10, U$1G$2.5V@1
- net GND: now also J3-1.S, U$2G$1.GND@3, U$2G$1.GND@4; no longer U$1G$2.GND@3, U$1G$2.GND@4
- net GND1: now also D1.A, D3.A; no longer D2.A, D4.A
- net LF_TX_UC: now also U$2G$2.PC6; no longer U$1G$3.PC6
- net SPI2_MISO: now also U$2G$1.PC2; no longer U$1G$2.PC2
- net SPI2_MOSI: now also U$2G$1.PC3; no longer U$1G$2.PC3
- net SPI2_SCK: now also U$2G$2.PB10@1; no longer U$1G$3.PB10@1
- net SPI2_SS: now also U$2G$1.PC1@1; no longer U$1G$2.PC1@1
- net SPI3_MISO: now also Q2.S, R12.1, U$2G$1.PC11; no longer Q1.S, R11.1, U$1G$2.PC11
- net SPI3_MISO_EXT: now also R11.1; no longer R12.1
- net SPI3_MOSI: now also Q4.S, R14.1, U$2G$1.PC12; no longer Q3.S, R9.1, U$1G$2.PC12
- net SPI3_MOSI_EXT: now also R9.1; no longer R10.1
- net SPI3_SCK: now also Q1.S, R10.1, U$2G$2.PB12; no longer Q2.S, R13.1, U$1G$3.PB12
- net SPI3_SS: now also Q3.S, R17.1, U$2G$2.PC9; no longer Q4.S, R15.1, U$1G$3.PC9
- net SPI3_SS_EXT: now also R13.1; no longer R14.1
- net SPI3_SS_EXT1: now also R15.1; no longer R16.1
- net USART1_RX: now also U$2G$2.PA10@1; no longer U$1G$1.PA10@10
- net USART1_TX: now also U$2G$2.PA9@1; no longer U$1G$1.PA9@10
- net VCC: now also R10.2, R12.2, R14.2, R17.2, U$2G$1.3V3@1; no longer R11.2, R13.2, R15.2, R9.2, U$1G$2.3V3@1
