File: gs_hab_mainboard/gs_mainboard_2.sch (EAGLE design)
At the start: 40 parts, among them IC1 LM4040/385 (2.5V), IC2 LM358D, J2 Storm Det, J6 LF Comm, J7 HF Comm, J8 Weather stat., J9 Ext 5V, Q1 BSS138, Q2 BSS138, Q3 BSS138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

Commit message: final, after another review
Parts:
- J8: value Weather stat. -> Weather st.
Changed lines of the file:
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@@
 <part name="J6" library="EP_molex_6410_7395" deviceset="22-?-05" device="05-7058" value="LF Comm"/>
 <part name="J7" library="EP_molex_6410_7395" deviceset="22-?-05" device="05-7058" value="HF Comm"/>
-<part name="J8" library="EP_molex_6410_7395" deviceset="22-?-07" device="05-7078" value="Weather stat."/>
+<part name="J8" library="EP_molex_6410_7395" deviceset="22-?-07" device="05-7078" value="Weather st."/>
 <part name="J9" library="EP_molex_6410_7395" deviceset="22-?-03" device="05-7038" value="Ext 5V"/>
 <part name="J2" library="EP_molex_6410_7395" deviceset="22-?-03" device="05-7038" value="Storm Det"/>
