File: gs_hab_mainboard/gs_mainboard_3.sch (EAGLE design)
At the start: 40 parts, among them IC1 LM4040/385 (2.5V), IC2 LM358D, J1 Weather st., J2 Storm Det, J6 LF Comm, J7 HF Comm, J9 Ext 5V, Q1 BSS138, Q2 BSS138, Q3 BSS138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

Commit message: corrected gerbers, cleaned schematics, added documnetation
Other:
- note added: "HF communication (IO)"
- note added: "LF transmitter"
- note added: "Storm detector and LF receiver"
- note added: "V_storm = analog 0..9V"
- note added: "Weather station (IO)"
- note added: "supply@5V uart@3.3V"
- note removed: "Storm detector = Analog 0..9V"
- note removed: "na PCB dodac mocowanie kabla usb"
- note removed: "wątpliwości co do odbioru radia?"
- note removed: "zasilanie z 5V, ale piny ogolnie jest na 3,3V"
- moved on the sheet: C2, J1-1, J1-2, J1-3, J1-4, J1-5, J1-6, J1-7, J1-8, J7-1, J7-2, J7-3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
