File: beacon_power_management/PMS.brd (EAGLE design)
At the start: 55.8 x 98.5 mm, 52 parts, among them IC2 M24M02-DR, IC3 LM258, IC4 LM258, J1 SOLARP1, J10 VBAT2_CHRG, J11 PLED1, J12 PLED2, J13 PLED3, J14 DWM, J2 SOLARP2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

Commit message: really final projects, added gerber files
Parts:
- L1, L2: device resistor:L2012C -> resistor:L3225M
Other:
- board text added: "."

Commit message: corrected gerbers, cleaned schematics, added documnetation
Changed lines of the file:
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@@
 <layer number="19" name="Unrouted" color="6" fill="1" visible="yes" active="yes"/>
 <layer number="20" name="Dimension" color="24" fill="1" visible="yes" active="yes"/>
-<layer number="21" name="tPlace" color="7" fill="1" visible="yes" active="yes"/>
-<layer number="22" name="bPlace" color="7" fill="1" visible="yes" active="yes"/>
+<layer number="21" name="tPlace" color="7" fill="1" visible="no" active="yes"/>
+<layer number="22" name="bPlace" color="7" fill="1" visible="no" active="yes"/>
 <layer number="23" name="tOrigins" color="15" fill="1" visible="yes" active="yes"/>
 <layer number="24" name="bOrigins" color="15" fill="1" visible="yes" active="yes"/>
@@
 <wire x1="76.25" y1="112.25" x2="20.5" y2="112.25" width="0" layer="20"/>
 <wire x1="20.5" y1="112.25" x2="20.5" y2="13.75" width="0" layer="20"/>
-<text x="34.5" y="70" size="1.016" layer="25" rot="MR0">+</text>
+<text x="35.41" y="71.33" size="1.016" layer="26" rot="MR270">+</text>
 <wire x1="76.25" y1="13.75" x2="20.5" y2="13.75" width="0" layer="20"/>
 <text x="33.23" y="15.008" size="1.27" layer="25" font="vector" ratio="15">PMS Shield
