File: beacon_power_management/PMS.sch (EAGLE design)
At the start: 52 parts, among them IC2 M24M02-DR, IC3 LM258, IC4 LM258, J1 SOLARP1, J10 VBAT2_CHRG, J11 PLED1, J12 PLED2, J13 PLED3, J14 DWM, J2 SOLARP2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

Commit message: really final projects, added gerber files
Parts:
- L1, L2: device resistor:L-USL2012C -> resistor:L-USL3225M

Commit message: corrected gerbers, cleaned schematics, added documnetation
Other:
- note added: "C3 = EEUFC1J101L"
- note added: "C4 = EEUFC1J101L"
- note removed: "Kondensatory do paneli - EEUFC1J101L"
- moved on the sheet: C1, C2, C3, C4, D1, D2, IC1, IC2, IC2P, IC3B, IC4A, IC4B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
