File: dwm_shield/DWM_shield.sch (EAGLE design)
At the start: 34 parts, among them IC1 DWM1000, IC2 LD1117S33C, J2 ARDU_COM, Q1 BSS138, Q2 BSS138, Q3 BSS138, Q4 BSS138, Q5 BSS138, Q6 BSS138

Commit message: corrected gerbers, cleaned schematics, added documnetation
Other:
- note added: "Arduino (IO)"
- note added: "Level shifters for IO"
- note added: "Power supply"
- moved on the sheet: C1, C2, C3, C4, D1, D2, D3, D4, IC1, IC2, J2-2, J2-3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
